Commit message: update: 360° lidar migration, urdf model update, slam params tuning

File: my_robot_description/urdf/xiaoche_hardware.ros2_control.xacro (robot description, xacro)
@@ -1,25 +1,23 @@
 <?xml version="1.0"?>
 <robot xmlns:xacro="http://www.ros.org/wiki/xacro">
-    <ros2_control name="MobileBase" type="system">
-        <hardware>
-            <!-- 使用实际硬件接口插件 -->
-            <plugin>mobile_base_hardware/MobileBaseHardwareInterface</plugin>
-            <param name="can_interface">can0</param>
-            <param name="node_id">1</param>
-            <param name="accel_time_ms">1000</param>
-            <param name="decel_time_ms">800</param>
-            <param name="torque_slope_ma_s">500</param>
-        </hardware>
-        <!-- 左右驱动轮 -->
-        <joint name="base_left_wheel_joint">
-            <command_interface name="velocity"/>
-            <state_interface name="position"/>
-            <state_interface name="velocity"/>
-        </joint>
-        <joint name="base_right_wheel_joint">
-            <command_interface name="velocity"/>
-            <state_interface name="position"/>
-            <state_interface name="velocity"/>
-        </joint>
-    </ros2_control>
+  <ros2_control name="MobileBase" type="system">
+    <hardware>
+      <plugin>mobile_base_hardware/MobileBaseHardwareInterface</plugin>
+      <param name="can_interface">can0</param>
+      <param name="node_id">1</param>
+      <param name="accel_time_ms">1000</param>
+      <param name="decel_time_ms">800</param>
+      <param name="torque_slope_ma_s">500</param>
+    </hardware>
+    <joint name="base_left_wheel_joint">
+      <command_interface name="velocity"/>
+      <state_interface name="position"/>
+      <state_interface name="velocity"/>
+    </joint>
+    <joint name="base_right_wheel_joint">
+      <command_interface name="velocity"/>
+      <state_interface name="position"/>
+      <state_interface name="velocity"/>
+    </joint>
+  </ros2_control>
 </robot>

File: my_robot_description/urdf/xiaoche_hardware.urdf.xacro (robot description, xacro)
@@ -1,7 +1,7 @@
 <?xml version="1.0"?>
 <robot xmlns:xacro="http://www.ros.org/wiki/xacro" name="xiaoche">
-    <!-- 引入底盘结构（已包含激光雷达） -->
-    <xacro:include filename="$(find my_robot_description)/urdf/xiaoche_shiyan_control.urdf.xacro"/>
-    <!-- 引入ros2_control配置 -->
-    <xacro:include filename="$(find my_robot_description)/urdf/xiaoche_hardware.ros2_control.xacro"/>
+  <!-- Robot structure exported from the latest URDF data. -->
+  <xacro:include filename="$(find my_robot_description)/urdf/xiaoche_shiyan_control.urdf.xacro"/>
+  <!-- ros2_control hardware/controller interfaces for the mobile base. -->
+  <xacro:include filename="$(find my_robot_description)/urdf/xiaoche_hardware.ros2_control.xacro"/>
 </robot>

File: my_robot_description/urdf/xiaoche_shiyan_control.urdf.xacro (robot description, xacro)
@@ -1,6 +1,7 @@
-<?xml version="1.0"?>
+<?xml version="1.0" encoding="utf-8"?>
+<!-- This URDF was automatically created by SolidWorks to URDF Exporter! Originally created by Stephen Brawner (brawner@gmail.com)
+     Commit Version: 1.5.1-0-g916b5db  Build Version: 1.5.7152.31018
+     For more information, please see http://wiki.ros.org/sw_urdf_exporter -->
 <robot xmlns:xacro="http://www.ros.org/wiki/xacro">
-  <!-- 使用file://绝对路径以解决Gazebo Harmonic的mesh加载问题 -->
-  <xacro:property name="mesh_prefix" value="package://my_robot_description" />
   <link name="base_footprint">
   </link>
@@ -8,5 +9,5 @@
     <parent link="base_footprint" />
     <child link="base_link" />
-    <origin xyz="0 0 0.2437139748" rpy="0 0 0" />
+    <origin xyz="0 0 0" rpy="0 0 0" />
   </joint>
   <link
@@ -14,37 +15,37 @@
     <inertial>
       <origin
-        xyz="0.012839 0.0021524 0.018198"
-        rpy="0 0 0" />
-      <mass
-        value="112.9" />
-      <inertia
-        ixx="0.65063"
-        ixy="0.00059995"
-        ixz="3.0503E-05"
-        iyy="0.6847"
-        iyz="-2.6829E-06"
-        izz="1.2368" />
-    </inertial>
-    <visual>
-      <origin
-        xyz="0 0 0"
-        rpy="0 0 0" />
-      <geometry>
-        <mesh
-          filename="${mesh_prefix}/meshes/base_link.STL" />
-      </geometry>
-      <material
-        name="">
-        <color
-          rgba="0.52941 0.54902 0.54902 1" />
-      </material>
-    </visual>
-    <collision>
-      <origin
-        xyz="0 0 0"
-        rpy="0 0 0" />
-      <geometry>
-        <mesh
-          filename="${mesh_prefix}/meshes/base_link.STL" />
+        xyz="0.00291971353695461 -0.00137055396386509 0.247093009152642"
+        rpy="0 0 0" />
+      <mass
+        value="5.71330094696822" />
+      <inertia
+        ixx="0.0451901760143035"
+        ixy="0.000112861110087808"
+        ixz="-3.74742789795674E-06"
+        iyy="0.0464614381420226"
+        iyz="-2.24460034513834E-06"
+        izz="0.0750479340967576" />
+    </inertial>
+    <visual>
+      <origin
+        xyz="0 0 0"
+        rpy="0 0 0" />
+      <geometry>
+        <mesh
+          filename="package://my_robot_description/meshes/base_link.STL" />
+      </geometry>
+      <material
+        name="">
+        <color
+          rgba="1 1 1 1" />
+      </material>
+    </visual>
+    <collision>
+      <origin
+        xyz="0 0 0"
+        rpy="0 0 0" />
+      <geometry>
+        <mesh
+          filename="package://my_robot_description/meshes/base_link.STL" />
       </geometry>
     </collision>
@@ -54,37 +55,37 @@
     <inertial>
       <origin
-        xyz="3.98238914067761E-10 1.61235126279469E-06 0.000174863057808228"
-        rpy="0 0 0" />
-      <mass
-        value="8.11370268019001" />
-      <inertia
-        ixx="0.0137875502161336"
-        ixy="-1.19298410300165E-09"
-        ixz="-1.55305504435677E-08"
-        iyy="0.0137874200888679"
-        iyz="-8.18605700359875E-07"
-        izz="0.0257560643934428" />
-    </inertial>
-    <visual>
-      <origin
-        xyz="0 0 0"
-        rpy="0 0 0" />
-      <geometry>
-        <mesh
-          filename="${mesh_prefix}/meshes/left_wheel_link.STL" />
-      </geometry>
-      <material
-        name="">
-        <color
-          rgba="0.752941176470588 0.752941176470588 0.752941176470588 1" />
-      </material>
-    </visual>
-    <collision>
-      <origin
-        xyz="0 0 0"
-        rpy="0 0 0" />
-      <geometry>
-        <mesh
-          filename="${mesh_prefix}/meshes/left_wheel_link.STL" />
+        xyz="1.9705E-06 4.2704E-08 -0.00091033"
+        rpy="0 0 0" />
+      <mass
+        value="0.94197" />
+      <inertia
+        ixx="0.0015823"
+        ixy="-3.7887E-10"
+        ixz="1.0322E-07"
+        iyy="0.0015823"
+        iyz="3.8949E-11"
+        izz="0.0029546" />
+    </inertial>
+    <visual>
+      <origin
+        xyz="0 0 0"
+        rpy="0 0 0" />
+      <geometry>
+        <mesh
+          filename="package://my_robot_description/meshes/left_wheel_link.STL" />
+      </geometry>
+      <material
+        name="">
+        <color
+          rgba="1 1 1 1" />
+      </material>
+    </visual>
+    <collision>
+      <origin
+        xyz="0 0 0"
+        rpy="0 0 0" />
+      <geometry>
+        <mesh
+          filename="package://my_robot_description/meshes/left_wheel_link.STL" />
       </geometry>
     </collision>
@@ -94,6 +95,6 @@
     type="continuous">
     <origin
-      xyz="0 0.1776 -0.15721"
-      rpy="1.5708 1.0806 3.1416" />
+      xyz="-0.0047976 0.1766 0.06604"
+      rpy="1.5708 0 3.1416" />
     <parent
       link="base_link" />
@@ -107,37 +108,37 @@
     <inertial>
       <origin
-        xyz="-6.17699953686657E-11 -1.61235131579396E-06 0.00017486305780906"
-        rpy="0 0 0" />
-      <mass
-        value="8.11370268019039" />
-      <inertia
-        ixx="0.0137875502166307"
-        ixy="-1.16582667763441E-09"
-        ixz="1.53597241964897E-08"
-        iyy="0.0137874200883763"
-        iyz="8.18608923761562E-07"
-        izz="0.0257560643934482" />
-    </inertial>
-    <visual>
-      <origin
-        xyz="0 0 0"
-        rpy="0 0 0" />
-      <geometry>
-        <mesh
-          filename="${mesh_prefix}/meshes/right_wheel_link.STL" />
-      </geometry>
-      <material
-        name="">
-        <color
-          rgba="0.752941176470588 0.752941176470588 0.752941176470588 1" />
-      </material>
-    </visual>
-    <collision>
-      <origin
-        xyz="0 0 0"
-        rpy="0 0 0" />
-      <geometry>
-        <mesh
-          filename="${mesh_prefix}/meshes/right_wheel_link.STL" />
+        xyz="-1.9705E-06 -4.2704E-08 -0.00091033"
+        rpy="0 0 0" />
+      <mass
+        value="0.94197" />
+      <inertia
+        ixx="0.0015823"
+        ixy="-3.7887E-10"
+        ixz="-1.0322E-07"
+        iyy="0.0015823"
+        iyz="-3.8949E-11"
+        izz="0.0029546" />
+    </inertial>
+    <visual>
+      <origin
+        xyz="0 0 0"
+        rpy="0 0 0" />
+      <geometry>
+        <mesh
+          filename="package://my_robot_description/meshes/right_wheel_link.STL" />
+      </geometry>
+      <material
+        name="">
+        <color
+          rgba="1 1 1 1" />
+      </material>
+    </visual>
+    <collision>
+      <origin
+        xyz="0 0 0"
+        rpy="0 0 0" />
+      <geometry>
+        <mesh
+          filename="package://my_robot_description/meshes/right_wheel_link.STL" />
       </geometry>
     </collision>
@@ -147,6 +148,6 @@
     type="continuous">
     <origin
-      xyz="0 -0.177600000000001 -0.157213947478889"
-      rpy="-1.5707963267949 0.00880119302616804 3.14159265358979" />
+      xyz="-0.0047976 -0.1766 0.06604"
+      rpy="1.5708 0 0" />
     <parent
       link="base_link" />
@@ -160,45 +161,45 @@
     <inertial>
       <origin
-        xyz="-0.000798649254042161 -3.09358095402987E-05 0.00537427843767044"
-        rpy="0 0 0" />
-      <mass
-        value="0.458153593425532" />
-      <inertia
-        ixx="3.44259629214186E-05"
-        ixy="1.05451170440238E-08"
-        ixz="-6.64868186292802E-07"
-        iyy="0.000265470306492972"
-        iyz="-4.33797609906098E-08"
-        izz="0.000272641640441728" />
-    </inertial>
-    <visual>
-      <origin
-        xyz="0 0 0"
-        rpy="0 0 0" />
-      <geometry>
-        <mesh
-          filename="${mesh_prefix}/meshes/camera_link.STL" />
-      </geometry>
-      <material
-        name="">
-        <color
-          rgba="0.529411764705882 0.549019607843137 0.549019607843137 1" />
-      </material>
-    </visual>
-    <collision>
-      <origin
-        xyz="0 0 0"
-        rpy="0 0 0" />
-      <geometry>
-        <mesh
-          filename="${mesh_prefix}/meshes/camera_link.STL" />
-      </geometry>
-    </collision>
-  </link>
-  <joint
-    name="base_camera_joint"
-    type="fixed">
-    <origin
-      xyz="0.2288 -5.2887E-05 0.044786"
+        xyz="-0.00074797 -2.9971E-05 -0.015771"
+        rpy="0 0 0" />
+      <mass
+        value="0.058736" />
+      <inertia
+        ixx="4.4134E-06"
+        ixy="1.6512E-09"
+        ixz="-8.5022E-08"
+        iyy="3.4033E-05"
+        iyz="-5.5548E-09"
+        izz="3.4952E-05" />
+    </inertial>
+    <visual>
+      <origin
+        xyz="0 0 0"
+        rpy="0 0 0" />
+      <geometry>
+        <mesh
+          filename="package://my_robot_description/meshes/camera_link.STL" />
+      </geometry>
+      <material
+        name="">
+        <color
+          rgba="1 1 1 1" />
+      </material>
+    </visual>
+    <collision>
+      <origin
+        xyz="0 0 0"
+        rpy="0 0 0" />
+      <geometry>
+        <mesh
+          filename="package://my_robot_description/meshes/camera_link.STL" />
+      </geometry>
+    </collision>
+  </link>
+  <joint
+    name="camera_joint"
+    type="fixed">
+    <origin
+      xyz="0.24835 0 0.27404"
       rpy="-1.5708 0 -1.5708" />
     <parent
@@ -213,46 +214,46 @@
     <inertial>
       <origin
-        xyz="-0.00250773388882672 3.90192185333316E-05 0.00570928899555997"
-        rpy="0 0 0" />
-      <mass
-        value="0.291977008093007" />
-      <inertia
-        ixx="0.000218819937566453"
-        ixy="6.68201015277679E-07"
-        ixz="-8.35224514646861E-06"
-        iyy="0.000262184949456141"
-        iyz="1.29957954178652E-07"
-        izz="0.000351682847727596" />
-    </inertial>
-    <visual>
-      <origin
-        xyz="0 0 0"
-        rpy="0 0 0" />
-      <geometry>
-        <mesh
-          filename="${mesh_prefix}/meshes/front_lidar_link.STL" />
-      </geometry>
-      <material
-        name="">
-        <color
-          rgba="0.376470588235294 0.376470588235294 0.376470588235294 1" />
-      </material>
-    </visual>
-    <collision>
-      <origin
-        xyz="0 0 0"
-        rpy="0 0 0" />
-      <geometry>
-        <mesh
-          filename="${mesh_prefix}/meshes/front_lidar_link.STL" />
-      </geometry>
-    </collision>
-  </link>
-  <joint
-    name="base_front_lidar_joint"
-    type="fixed">
-    <origin
-      xyz="0.1975 0 0.11518"
-      rpy="0 0 0.015558" />
+        xyz="-0.0035782 1.6334E-09 0.011632"
+        rpy="0 0 0" />
+      <mass
+        value="0.037432" />
+      <inertia
+        ixx="2.8051E-05"
+        ixy="8.4886E-11"
+        ixz="-1.071E-06"
+        iyy="3.3615E-05"
+        iyz="9.6473E-14"
+        izz="4.5086E-05" />
+    </inertial>
+    <visual>
+      <origin
+        xyz="0 0 0"
+        rpy="0 0 0" />
+      <geometry>
+        <mesh
+          filename="package://my_robot_description/meshes/front_lidar_link.STL" />
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